File: hardware/bdkb40.kicad_pcb (KiCad board)
At the start: 2 copper layers, 229.6 x 77.2 mm, 122 parts, among them J2 78171-0002, J4 SWD, J5 UART, J6 78171-0004, SW1 RST, SW2 FRST, SW3 DFU, SW4 SW_SP3T, U2 BQ24075, U3 MAX17048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

Commit message: pcb design move to hardware folder
Routing:
- net c01: track 149.0 -> 145.4 mm
- net c00: track 167.7 -> 164.3 mm
- net Net-(D25-A): track 4.39 -> 5.05 mm
- net r3: track 320.6 -> 320.0 mm

Commit message: update pcb
Parts:
- moved LED1 0.26 mm to (611.4, 90.4)
Routing:
- net c06: track 140.6 -> 149.2 mm, vias 0 -> 2
- net Net-(U4-P0.10/NFC2): track 167.3 -> 165.4 mm
- net Net-(U4-P1.06): track 165.3 -> 164.5 mm
- net Net-(U4-P0.09/NFC1): track 158.1 -> 157.5 mm
- net GND: track 321.7 -> 321.1 mm, vias 51 -> 43
- net SWDCLK: track 23.9 -> 24.6 mm

Commit message: update pcd
Parts:
- added ?: , , F.Cu at (193.5, 121.1)
- added ?: , , F.Cu at (226.8, 73.5)
- added ?: , , F.Cu at (55.3, 111.6)
- added ?: , , F.Cu at (131.5, 73.5)
- added ?: , , F.Cu at (55.3, 73.5)
- added ?: , , F.Cu at (98.2, 121.1)
- added ?: , , F.Cu at (236.3, 111.6)
- moved MX41 510.7 mm to (167.3, 121.1)
- moved C13 510.5 mm to (139.7, 109.0)
- moved C2 510.5 mm to (153.9, 107.2)
- moved C3 510.5 mm to (155.2, 107.2)
- moved D11 510.5 mm to (224.5, 67.3)
- moved D13 510.5 mm to (36.4, 86.3)
- moved D14 510.5 mm to (57.8, 86.3)
- moved D16 510.5 mm to (95.9, 86.3)
- moved D19 510.5 mm to (153.1, 86.3)
- moved D21 510.5 mm to (191.2, 86.3)
- moved D23 510.5 mm to (236.4, 86.3)
- moved D3 510.5 mm to (72.1, 67.3)
- moved D33 510.5 mm to (199.8, 95.4)
- moved D37 510.5 mm to (36.4, 124.4)
- moved D42 510.5 mm to (197.6, 114.8)
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
Commit message: update fabrication info
Parts:
- removed ? (x7): , 
- SW1, SW2, SW3: footprint PCM_marbastlib-various:SW_T1A2QR -> Button_Switch_SMD:SW_SPST_TS-1088-xR025
- SW4: value SW_SP3T -> SW_SP3T_TA3517A1
- moved J4 7.12 mm to (172.4, 128.7)
- moved SW1 5.76 mm to (166.0, 129.2)
- moved SW3 3.20 mm to (160.1, 129.2)
- moved SW2 0.61 mm to (154.0, 129.2)
Routing:
- net r3: track 319.8 -> 348.3 mm
- net SWDIO: track 24.4 -> 31.1 mm
- net SWDCLK: track 24.6 -> 31.1 mm
- net RST: track 25.1 -> 30.4 mm
- net c06: track 148.9 -> 145.2 mm
- net GND: track 321.1 -> 324.8 mm, vias 43 -> 36
- net c01: track 145.4 -> 149.0 mm
- net c00: track 164.3 -> 167.7 mm
- net DFU: track 17.1 -> 19.9 mm
- net FRST: track 12.6 -> 14.0 mm
- net Net-(U4-P0.10/NFC2): track 165.4 -> 164.4 mm, vias 0 -> 2
- net Net-(U4-P1.06): track 164.5 -> 164.1 mm, vias 0 -> 2
- net Net-(U4-P0.09/NFC1): track 157.5 -> 157.4 mm, vias 0 -> 2
