File: hardware/bdkb40.kicad_sch (KiCad schematic)
At the start: 125 parts, among them J2 78171-0002, J3 TC2030_SWD, J4 SWD, J5 UART, J6 78171-0004, SW1 RST, SW2 FRST, SW3 DFU, SW4 SW_SP3T, U2 BQ24075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

Commit message: update fabrication info
Parts:
- SW1, SW2, SW3: footprint PCM_marbastlib-various:SW_T1A2QR -> Button_Switch_SMD:SW_SPST_TS-1088-xR025; LCSC C100056 -> C720477
- SW4: value SW_SP3T -> SW_SP3T_TA3517A1; LCSC (none) -> C514001
Changed lines of the file:
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@@
 			)
 		)
-		(property "Footprint" "PCM_marbastlib-various:SW_T1A2QR"
+		(property "Footprint" "Button_Switch_SMD:SW_SPST_TS-1088-xR025"
 			(at 106.68 -162.56 0)
 			(effects
@@
 			)
 		)
-		(property "LCSC" "C100056"
+		(property "LCSC" "C720477"
 			(at 101.6 -162.56 0)
 			(effects
@@
 			)
 		)
-		(property "Footprint" "PCM_marbastlib-various:SW_T1A2QR"
+		(property "Footprint" "Button_Switch_SMD:SW_SPST_TS-1088-xR025"
 			(at 85.09 -162.56 0)
 			(effects
@@
 			)
 		)
-		(property "LCSC" "C100056"
+		(property "LCSC" "C720477"
 			(at 80.01 -162.56 0)
 			(effects
@@
 			)
 		)
-		(property "Footprint" "PCM_marbastlib-various:SW_T1A2QR"
+		(property "Footprint" "Button_Switch_SMD:SW_SPST_TS-1088-xR025"
 			(at 96.52 -162.56 0)
 			(effects
@@
 			)
 		)
-		(property "LCSC" "C100056"
+		(property "LCSC" "C720477"
 			(at 91.44 -162.56 0)
 			(effects
@@
 			)
 		)
-		(property "Value" "SW_SP3T"
+		(property "Value" "SW_SP3T_TA3517A1"
 			(at 59.69 -144.78 0)
 			(effects
@@
 			(effects
 				(font
+					(size 1.27 1.27)
+				)
+				(hide yes)
+			)
+		)
+		(property "LCSC" "C514001"
+			(at 59.69 -147.32 0)
+			(effects
+				(font
